File: Sharkbyte-Debugger-Mini.kicad_sch (KiCad schematic)
At the start: 155 parts, among them J2 Conn_01x15_Pin, Q1 SS8050 200-350, Q2 AO3401A, U1 STM32G474CBTx, U10 TCAN1042VDRQ1, U11 HC-TYPE-C-16P-CB1_6, U12 STUSB4500QTR, U13 STL6P3LLH6-TP, U14 STL6P3LLH6-TP, U15 TPS63070RNMR, U16 MDE0518-2R2M, U17 MDE0518-2R2M, U18 TPS63070RNMR, U2 REF3030, U3 MDE0518-2R2M, U4 W25Q128JVSIQTR, U5 CC6920SO-20A, U6 TPS55287RYQR, U7 TLV9361IDBVR, U8 ACS712xLCTR-05B, U9 TLV9361IDBVR, Y1 Crystal_GND24

Commit message: layout
Parts:
- removed C26, C27: 100nF, PCM_JLCPCB:C_0402, symbol Device:C
- removed D3: BAV99, Package_TO_SOT_SMD:SOT-23, symbol Diode:BAV99
- removed Q2: AO3401A, PCM_JLCPCB:Q_SOT-23, symbol PCM_JLCPCB-Transistors:PMOS,AO3401A
- removed R6: 100R, PCM_JLCPCB:R_0402, symbol Device:R
- removed R7, R8: 10K, PCM_JLCPCB:R_0402, symbol Device:R
- removed U5: CC6920SO-20A, JLC_PARTS:SOP-8_L5.0-W4.0-P1.27-LS6.2-BL, symbol JLC_PARTS:CC6920SO-20A
- added C76, C77, C78: 100nF, PCM_JLCPCB:C_0402, symbol Device:C
- added D9: BAV99, Package_TO_SOT_SMD:SOT-23, symbol Diode:BAV99
- added Q3: SS8050 200-350, PCM_JLCPCB:Q_SOT-23, symbol PCM_JLCPCB-Transistors:NPN,SS8050 200-350
- added Q4: AO3401A, PCM_JLCPCB:Q_SOT-23, symbol PCM_JLCPCB-Transistors:PMOS,AO3401A
- added R19: 100R, PCM_JLCPCB:R_0402, symbol Device:R
- added R50, R51, R52: 120R, PCM_JLCPCB:R_0402, symbol Device:R
- added R53, R54, R55: 10K, PCM_JLCPCB:R_0402, symbol Device:R
- added U19: ACS712xLCTR-05B, Package_SO:SOIC-8_3.9x4.9mm_P1.27mm, symbol Sensor_Current:ACS712xLCTR-05B
- C73, C74: footprint PCM_JLCPCB:C_0402 -> PCM_JLCPCB:C_0603
- R3: footprint PCM_JLCPCB:R_0805 -> PCM_JLCPCB:R_0603
Connections:
- net +3.3V: now also C14.2, J1.9 (VDD), J2.9 (Pin_9), D9.2 (A), R53.1; no longer C14.1, C15.2, J1.7 (GND), J1.8 (VSS), J2.1 (Pin_1), R22.2
- net +5V: now also C77.1, U19.8 (VCC)
- net AMMETER_ADC: now also C76.1, R19.1
- net AMMETER_IN: now also J2.4 (Pin_4), U19.1 (IP+), U19.2 (IP+); no longer J2.6 (Pin_6)
- net AMMETER_OUT: now also J2.3 (Pin_3), U19.3 (IP-), U19.4 (IP-); no longer J2.7 (Pin_7)
- net CANH: now also R51.1, R52.1
- net CANL: now also R50.2
- net CAN_R_GPIO: now also U1.2 (PC13), R54.1; no longer R22.1
- net CS#: now also U1.4 (PC15); no longer U1.3 (PC14)
- net FUNCTION_GEN_OUT: now also J2.6 (Pin_6); no longer J2.11 (Pin_11)
- net GND: now also C14.1, C15.2, J1.7 (GND), J1.8 (VSS), J2.1 (Pin_1), J2.8 (Pin_8), C76.2, C77.2, C78.2, D9.1 (K), Q3.2 (E), Q4.3 (D), R55.1, U19.5 (GND); no longer J2.5 (Pin_5), J2.9 (Pin_9)
- net NRST: now also J2.10 (Pin_10); no longer J2.2 (Pin_2)
- net OHMMETER_ADC: now also J2.7 (Pin_7); no longer J2.8 (Pin_8)
- net PSU_CON: now also J2.2 (Pin_2); no longer J2.12 (Pin_12)
- net RES#: now also U1.3 (PC14); no longer U1.2 (PC13)
- net SCOPE_OUT: now also J2.5 (Pin_5); no longer J2.10 (Pin_10)
- net SWCLK: now also J2.11 (Pin_11); no longer J2.3 (Pin_3)
- net SWDIO: now also J2.12 (Pin_12); no longer J2.4 (Pin_4)
- net USB_PD_RESET: now also U1.29 (PB15); no longer U1.4 (PC15)
- net VPSU_ADC: now also C37.1, R17.1; no longer D5.3 (K), R15.1, R16.2
- net at U8.7 (VIOUT): now also R15.2; no longer R17.2
- net at R21.1: now also Q4.2 (S), R50.1, R51.2, R52.2
- new net: C78.1, U19.6 (FILTER)
- new net: R22.2, U19.7 (VIOUT)
- new net: Q3.3 (C), Q4.1 (G), R53.2
- new net: D9.3 (K), R19.2, R22.1, R55.2
- new net: Q3.1 (B), R54.2
- new net: D5.3 (K), R15.1, R16.2, R17.2
- no-connect marks 14 -> 12
Other:
- note added: "CAN Termination"
- note removed: "IN"
- note removed: "OUT"
- moved on the sheet: BUZ1, D1, D4, D5, Q1, R10, R11, R15, R16, R21, R23
