File: Sharkbyte-Debugger-Mini.kicad_pcb (KiCad board)
At the start: 4 copper layers, 80 x 60 mm, 155 parts, among them J2 Conn_01x15_Pin, Q1 SS8050 200-350, Q2 AO3401A, U1 STM32G474CBTx, U10 TCAN1042VDRQ1, U11 HC-TYPE-C-16P-CB1_6, U12 STUSB4500QTR, U13 STL6P3LLH6-TP, U14 STL6P3LLH6-TP, U15 TPS63070RNMR, U16 MDE0518-2R2M, U17 MDE0518-2R2M, U18 TPS63070RNMR, U2 REF3030, U3 MDE0518-2R2M, U4 W25Q128JVSIQTR, U5 CC6920SO-20A, U6 TPS55287RYQR, U7 TLV9361IDBVR, U8 ACS712xLCTR-05B, U9 TLV9361IDBVR, Y1 Crystal_GND24

Commit message: add zone fills
Routing:
- net Net-(U6-BOOT2): track 0.00 -> 0.97 mm
- net Net-(U6-BOOT1): track 0.00 -> 0.97 mm
- net Vin: vias 22 -> 41
- net Net-(U6-VOUT): vias 0 -> 8
- net GND: vias 15 -> 25
- added copper zone on F.Cu, net Net-(U6-SW1)
- added copper zone on F.Cu, net Net-(U6-SW2)
- added copper zone on In2.Cu, net Net-(U6-VOUT)

Commit message: layout
Parts:
- removed C26, C27: 100nF, PCM_JLCPCB:C_0402
- removed D3: BAV99, Package_TO_SOT_SMD:SOT-23
- removed Q2: AO3401A, PCM_JLCPCB:Q_SOT-23
- removed R6: 100R, PCM_JLCPCB:R_0402
- removed R7, R8: 10K, PCM_JLCPCB:R_0402
- removed U5: CC6920SO-20A, JLC_PARTS:SOP-8_L5.0-W4.0-P1.27-LS6.2-BL
- added C76: 100nF, PCM_JLCPCB:C_0402, F.Cu at (117.7, 123.5)
- added C77: 100nF, PCM_JLCPCB:C_0402, F.Cu at (116.3, 109.2)
- added C78: 100nF, PCM_JLCPCB:C_0402, F.Cu at (116.3, 107.0)
- added D9: BAV99, Package_TO_SOT_SMD:SOT-23, F.Cu at (119.5, 121.6)
- added Q3: SS8050 200-350, PCM_JLCPCB:Q_SOT-23, F.Cu at (121.8, 138.1)
- added Q4: AO3401A, PCM_JLCPCB:Q_SOT-23, F.Cu at (117.9, 138.1)
- added R19: 100R, PCM_JLCPCB:R_0402, F.Cu at (117.7, 122.7)
- added R50: 120R, PCM_JLCPCB:R_0402, F.Cu at (115.5, 139.0)
- added R51: 120R, PCM_JLCPCB:R_0402, F.Cu at (115.5, 137.2)
- added R52: 120R, PCM_JLCPCB:R_0402, F.Cu at (114.7, 137.2)
- added R53: 10K, PCM_JLCPCB:R_0402, F.Cu at (124.2, 137.2)
- added R54: 10K, PCM_JLCPCB:R_0402, F.Cu at (124.2, 139.1)
- added R55: 10K, PCM_JLCPCB:R_0402, F.Cu at (122.0, 122.5)
- added U19: ACS712xLCTR-05B, Package_SO:SOIC-8_3.9x4.9mm_P1.27mm, F.Cu at (120.5, 108.0)
- C73, C74: footprint PCM_JLCPCB:C_0402 -> PCM_JLCPCB:C_0603
- R18: footprint Resistor_SMD:R_0612_1632Metric -> Resistor_SMD:R_1225_3264Metric
- R3: footprint PCM_JLCPCB:R_0805 -> PCM_JLCPCB:R_0603
- moved C12 157.2 mm to (135.3, 131.9), turned to -90 degrees
- moved C14 156.6 mm to (138.7, 131.4), turned to 180 degrees
- moved C13 155.3 mm to (134.4, 131.9), turned to 90 degrees
- moved C15 154.0 mm to (136.8, 131.4)
- moved R1 150.9 mm to (145.6, 132.8), turned to 180 degrees
- moved C18 146.6 mm to (148.4, 131.6)
- moved C16 145.8 mm to (145.6, 131.6), turned to 180 degrees
- moved C45 142.0 mm to (110.3, 141.0), turned to 180 degrees
- moved R21 139.7 mm to (114.7, 139.0), turned to -90 degrees
- moved C44 138.9 mm to (106.3, 138.0), turned to 90 degrees
- moved R15 136.9 mm to (122.0, 124.3), turned to 90 degrees
- moved R16 136.9 mm to (122.0, 126.1), turned to 90 degrees
- moved R17 132.8 mm to (117.7, 126.3)
- moved R22 128.6 mm to (122.0, 120.6), turned to 90 degrees
- moved R10 127.7 mm to (117.3, 130.4), turned to 90 degrees
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Connections:
- C14 pad 1: +3.3V -> GND
- C14 pad 2: Net-(J1-VDD) -> +3.3V
- C15 pad 2: +3.3V -> GND
- C37 pad 1: Net-(C37-Pad1) -> /VPSU_ADC
- D5 pad 3: /VPSU_ADC -> Net-(D5-K-Pad3)
- J1 pad 7: +3.3V -> GND
- J1 pad 8: +3.3V -> GND
- J1 pad 9: Net-(J1-VDD) -> +3.3V
- J2 pad 1: +3.3V -> GND
- J2 pad 10: /SCOPE_OUT -> /NRST
- J2 pad 11: /FUNCTION_GEN_OUT -> /SWCLK
- J2 pad 12: /PSU_CON -> /SWDIO
- J2 pad 2: /NRST -> /PSU_CON
- J2 pad 3: /SWCLK -> /AMMETER_OUT
- J2 pad 4: /SWDIO -> /AMMETER_IN
- J2 pad 5: GND -> /SCOPE_OUT
- J2 pad 6: /AMMETER_IN -> /FUNCTION_GEN_OUT
- J2 pad 7: /AMMETER_OUT -> /OHMMETER_ADC
- J2 pad 8: /OHMMETER_ADC -> GND
- J2 pad 9: GND -> +3.3V
- R15 pad 1: /VPSU_ADC -> Net-(D5-K-Pad3)
- R15 pad 2: Net-(C37-Pad1) -> Net-(U8-VIOUT)
- R16 pad 2: /VPSU_ADC -> Net-(D5-K-Pad3)
- R17 pad 1: Net-(C37-Pad1) -> /VPSU_ADC
- R17 pad 2: Net-(U8-VIOUT) -> Net-(D5-K-Pad3)
- R22 pad 1: /CAN_R_GPIO -> Net-(D9-K-Pad3)
- R22 pad 2: +3.3V -> Net-(U19-VIOUT)
- U1 pad 2: /RES# -> /CAN_R_GPIO
- U1 pad 29: unconnected-(U1-PB15-Pad29) -> /USB_PD_RESET
- U1 pad 3: /CS# -> /RES#
- U1 pad 4: /USB_PD_RESET -> /CS#
Routing:
- net /OHMMETER_ADC: track 0.00 -> 72.8 mm, vias 0 -> 2
- net /SWDIO: track 0.00 -> 70.2 mm
- net /SWCLK: track 0.00 -> 70.1 mm
- net /NRST: track 1.49 -> 70.4 mm
- net /CANH: track 0.00 -> 53.1 mm
- net /CANL: track 0.00 -> 52.5 mm
- net /SPI1_SCK: track 0.00 -> 48.6 mm
- net /SPI1_MOSI: track 0.00 -> 48.0 mm, vias 0 -> 2
- net /FUNCTION_GEN_OUT: track 0.00 -> 46.5 mm
- net /D/C#: track 0.00 -> 44.0 mm
- net /RES#: track 0.00 -> 40.4 mm
- net /SCOPE_OUT: track 0.00 -> 39.8 mm
- net /CS#: track 0.00 -> 39.6 mm
- net Net-(U8-VIOUT): track 0.00 -> 26.6 mm, vias 0 -> 2
- net GND: track 36.8 -> 63.1 mm, vias 25 -> 40
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Other:
- board size 80 x 60 mm -> 100 x 60 mm

Commit message: silkscreen
Parts:
- added G***: LOGO, LOGO, F.Cu at (86.0, 143.0)
- moved BUZ1 14.2 mm to (96.0, 136.0)
- moved Q1 14.2 mm to (96.0, 131.0)
- moved D1 14.0 mm to (99.7, 136.0)
- moved R23 13.6 mm to (98.2, 131.0)
Routing:
- net GND: vias 40 -> 41
Other:
- board text added: "3.3V"
- board text added: "5V"
- board text added: "A IN"
- board text added: "A OUT"
- board text added: "CAN H"
- board text added: "CAN L"
- board text added: "FUNC GEN"
- board text added: "GND"
- board text added: "MINI"
- board text added: "NRST"
- board text added: "OSC"
- board text added: "PSU"
- board text added: "SHARKBYTE DEBUGGER"
- board text added: "SWCLK"
- board text added: "SWDIO"
- board text added: "Ω IN"
- board text added: "Ω OUT"
